Commit message: Absolute mess, but front roll, pitch calibration works and urdf read in-out feature added.

File: results/lidar_cali.urdf (robot description, URDF)
Before this commit: robot a2rl_vehicle, 20 links, 19 joints
Joints:
- joint lidar_front: origin xyz=2.319 0.00268 0.68636 rpy=-0.37546573 -1.5461567 -2.7650 -> xyz=2.3380647651400577 -0.004089855490104472 0.677756668759084 rpy=-1.9782950124124146 -1.5543739169082464 -1.1623295145423838
- joint os_lidar: origin xyz=4.446 0.02 1.347 rpy=-0.018569 0.01447 -0.014 -> xyz=4.529968444196393 0.02926975868023582 1.2734364056565288 rpy=-0.012537884392003169 0.0446295144171891 -0.016890939383730708

Commit message: Not clean, but ready for calibration pipeline

File: results/lidar_cali.urdf (robot description, URDF)
Before this commit: robot a2rl_vehicle, 20 links, 19 joints
Joints:
- joint lidar_front: origin xyz=2.3380647651400577 -0.004089855490104472 0.677756668759084 rpy=-1.9782950124124146 -1.5543739169082464 -1.1623295145423838 -> xyz=2.336705241335275 0.0007543215968829292 0.6777519765090311 rpy=-2.0885913100586677 -1.5616717557497841 -1.0520486075985627
- joint lidar_left: origin xyz=1.76349 0.12679 0.7449607 rpy=-1.7899759 -1.5592 0.7437 -> xyz=1.8245261897761837 0.15400269083897508 0.7501353479382715 rpy=-1.2731980578937063 -1.5333732668329811 0.2237643543565873
- joint lidar_right: origin xyz=1.7286966 -0.11475 0.76980 rpy=2.916668 -1.564541 -1.86865887 -> xyz=1.8005809754138709 -0.09108359263480835 0.7789440650815105 rpy=1.2679204454671196 -1.5439791881790497 -0.22372712722718577
- joint os_lidar: origin xyz=4.529968444196393 0.02926975868023582 1.2734364056565288 rpy=-0.012537884392003169 0.0446295144171891 -0.016890939383730708 -> xyz=4.527005984494918 0.0381238776416746 1.2774865063846736 rpy=-0.019665734979499142 0.042505344479095486 -0.01717760535525066

Commit message: all_to_ouster calibration added.

File: results/lidar_cali.urdf (robot description, URDF)
Before this commit: robot a2rl_vehicle, 20 links, 19 joints
Links:
- link vehicle: geometry collision box size=5.2359 1.9207 1.2; visual box size=0.05 20 1.0
Joints:
- joint lidar_front: origin xyz=2.336705241335275 0.0007543215968829292 0.6777519765090311 rpy=-2.0885913100586677 -1.5616717557497841 -1.0520486075985627 -> xyz=2.282044425255705 -0.010037285272872832 0.688588347963234 rpy=-0.3753947880849591 -1.5464300686008563 -2.7512553820799317
- joint lidar_left: origin xyz=1.8245261897761837 0.15400269083897508 0.7501353479382715 rpy=-1.2731980578937063 -1.5333732668329811 0.2237643543565873 -> xyz=1.7187824378187708 0.10566213121500106 0.7449181083792673 rpy=-1.8039286328831663 -1.5590780850698356 0.7715362457914557
- joint lidar_right: origin xyz=1.8005809754138709 -0.09108359263480835 0.7789440650815105 rpy=1.2679204454671196 -1.5439791881790497 -0.22372712722718577 -> xyz=1.6978671550274618 -0.13951367918263644 0.7729420430023692 rpy=2.897749946089405 -1.5643347082895986 -1.836301214659613
- joint os_lidar: origin xyz=4.527005984494918 0.0381238776416746 1.2774865063846736 rpy=-0.019665734979499142 0.042505344479095486 -0.01717760535525066 -> xyz=4.406907516948252 0.03574011377571041 1.3476021580750932 rpy=-0.018913256191144655 0.014561210282393544 -1.814395860259373e-06
